File: STM_TEST/STM_TEST.brd (EAGLE design)
At the start: 80 x 64.8 mm, 35 parts, among them U1 TPS2115APWR, U2 AZ1117EH-3.3TRG1, Y2 ECS-80-S-4X

Commit message: Yay CAN
Parts:
- added C5, C6: 4.7nF, SparkFun-Capacitors:0603
- added J2: (no value), SparkFun-Connectors:1X02
- added R10, R11, R14, R15: 60, SparkFun-Resistors:0603
- added R12, R13, R16, R17: 0, SparkFun-Resistors:0603
- moved R5 87.7 mm to (111.2, 80.0), turned to 90 degrees
- moved R6 82.4 mm to (106.7, 73.3), turned to 270 degrees
- moved CR1 5.61 mm to (107.2, 79.4)
Connections:
- removed net CS1: CR1.1, R5.2
- new net CAN_H: J2.2, R12.2, R16.2
- new net CAN_L: J2.1, R13.2, R17.2
- new net N$1: C5.2, R10.1, R11.2
- new net N$10: R14.2, R16.1
- new net N$4: R11.1, R13.1
- new net N$5: R10.2, R12.1
- new net N$8: C6.2, R14.1, R15.2
- new net N$9: R15.1, R17.1
- new net NSS: CR1.1, R5.2, U$2.PA4
- net GND: now also C5.1, C6.1
Routing:
- net NSS: track 0.00 -> 18.2 mm, vias 0 -> 2
- net +3V3: track 52.0 -> 65.6 mm
- net SCK: track 0.00 -> 12.2 mm
- net MOSI: track 0.00 -> 8.03 mm
- net MISO: track 0.00 -> 7.24 mm
- added copper zone on layer 1, net +3V3

Commit message: Board Layout
Parts:
- added C7: 100nF, SparkFun-Capacitors:0603
- added U$1: TCAN337D, PI_Shield_Library:TCAN337D
- moved R17 108.2 mm to (75.9, 79.5), turned to 90 degrees
- moved R16 104.5 mm to (74.2, 79.5), turned to 90 degrees
- moved R15 97.3 mm to (75.1, 74.9), turned to 180 degrees
- moved R14 95.8 mm to (75.1, 76.6)
- moved C6 89.6 mm to (75.1, 73.3), turned to 180 degrees
- moved R13 89.3 mm to (65.0, 79.5), turned to 90 degrees
- moved R12 86.6 mm to (66.8, 79.5), turned to 90 degrees
- moved C5 77.2 mm to (65.9, 73.3)
- moved R11 75.6 mm to (65.9, 74.9)
- moved R10 74.1 mm to (65.9, 76.6), turned to 180 degrees
- moved J2 68.8 mm to (70.5, 82.9), turned to 270 degrees
Connections:
- removed net CAN_RX: U$2.PA11
- removed net CAN_TX: U$2.PA12
- new net CAN_STM_RX: U$1.TXD, U$2.PA11
- new net CAN_STM_TX: U$1.RXD, U$2.PA12
- net +3V3: now also C7.1, U$1.VCC
- net CAN_H: now also U$1.CANH
- net CAN_L: now also U$1.CANL
- net GND: now also C7.2, U$1.GND
Routing:
- net CAN_L: track 0.00 -> 27.1 mm
- net CAN_H: track 0.00 -> 19.9 mm, vias 0 -> 1
- net CAN_STM_TX: track 0.00 -> 15.9 mm, vias 0 -> 2
- net CAN_STM_RX: track 0.00 -> 14.7 mm, vias 0 -> 2
- net N$4: track 0.00 -> 5.55 mm
- net N$9: track 0.00 -> 5.47 mm
- net +3V3: track 65.6 -> 69.3 mm, vias 3 -> 4
- net N$5: track 0.00 -> 3.61 mm
- net N$10: track 0.00 -> 3.39 mm
- net N$8: track 0.00 -> 3.30 mm
- net N$1: track 0.00 -> 3.30 mm

Commit message: things
Parts:
- removed R12, R13, R16, R17: 0, SparkFun-Resistors:0603
- removed R14, R15: 60, SparkFun-Resistors:0603
- added U$3: TCAN337D, PI_Shield_Library:TCAN337D
- added U$5: MCP2515, PI_Shield_Library:MCP2515
- C6: value 4.7nF -> 100nF
- moved C5 17.4 mm to (71.2, 89.8), turned to 180 degrees
- moved R11 14.2 mm to (71.2, 88.1), turned to 180 degrees
- moved R10 11.3 mm to (71.2, 86.5), turned to 0 degrees
- moved J2 7.42 mm to (75.1, 88.8)
- moved C6 4.74 mm to (75.7, 68.6)
Connections:
- removed net N$4: R11.1, R13.1
- removed net N$5: R10.2, R12.1
- new net CAN_PI_RX: U$3.TXD, U$5.RXCAN
- new net CAN_PI_TX: U$3.RXD, U$5.TXCAN
- new net N$11: U$5.CS
- net +3V3: now also C6.1, U$3.VCC
- net CAN_H: now also R10.2, U$3.CANH; no longer R12.2, R16.2
- net CAN_L: now also R11.1, U$3.CANL; no longer R13.2, R17.2
- net GND: now also C6.2, U$3.GND; no longer C6.1
- net N$10: now also U$5.SO; no longer R14.2, R16.1
- net N$8: now also U$5.SCK; no longer C6.2, R14.1, R15.2
- net N$9: now also U$5.SI; no longer R15.1, R17.1
Routing:
- net CAN_L: track 27.1 -> 6.18 mm
- net CAN_H: track 19.9 -> 5.88 mm, vias 1 -> 0
- net N$4: track 5.55 -> 0.00 mm
- net N$9: track 5.47 -> 0.00 mm
- net N$5: track 3.61 -> 0.00 mm
- net N$10: track 3.39 -> 0.00 mm
- net N$8: track 3.30 -> 0.00 mm

Commit message: reroute
Parts:
- added C10, C8, C9: 100nF, SparkFun-Capacitors:0603
- added C11: 18pF, SparkFun-Capacitors:0603
- added Y1: ECS-80-S-4X, ECS-80-S-4X:XTAL_ECS-80-S-4X
- C18: value 100nF -> 18pF
- moved RESET1 78.8 mm to (156.1, 104.0)
- moved R8 78.8 mm to (161.0, 106.2)
- moved C18 65.7 mm to (67.1, 136.7), flipped to the bottom, turned to 90 degrees
- moved C6 60.9 mm to (85.5, 128.7), flipped to the bottom, turned to 270 degrees
- moved U$3 59.8 mm to (88.5, 131.2), turned to 180 degrees
- moved U$5 57.5 mm to (55.4, 135.4), turned to 180 degrees
- moved C7 49.8 mm to (85.5, 136.3), turned to 90 degrees
- moved J2 48.4 mm to (80.5, 136.9)
- moved R10 48.4 mm to (76.7, 134.6)
- moved C5 48.4 mm to (76.7, 137.9)
- moved R11 48.4 mm to (76.7, 136.3)
- moved U$1 48.4 mm to (88.5, 137.4)
- moved J1 47.5 mm to (104.6, 83.6)
- moved R3 39.3 mm to (97.7, 85.5), flipped to the bottom, turned to 270 degrees
- moved R4 38.1 mm to (100.3, 85.5), flipped to the bottom, turned to 270 degrees
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Connections:
- removed net N$10: U$5.SO
- removed net N$11: U$5.CS
- removed net N$8: U$5.SCK
- removed net N$9: U$5.SI
- new net OSC1: C18.1, U$5.OSC1, Y1.2
- new net OSC2: C11.1, U$5.OSC2, Y1.1
- net +3V3: now also C8.1, C9.1, U$5.VDD
- net +3V3BU: now also SW2.2; no longer SW2.1
- net +3V3ROV: now also SW2.1; no longer SW2.2
- net CE0: now also U$5.CS
- net D0: now also R4.2, SW1.2; no longer R3.2, SW1.1
- net D1: now also R3.2, SW1.1; no longer R4.2, SW1.2
- net GND: now also C10.2, C11.2, C8.2, C9.2, U$5.VSS
- net MISO_PI: now also U$5.SO
- net MOSI_PI: now also U$5.SI
- net NRST: now also C10.1; no longer C18.1
- net SCLK_PI: now also U$5.SCK
Routing:
- net +3V3: track 69.3 -> 0.12 mm, vias 4 -> 0
- net NRST: track 31.1 -> 0.00 mm, vias 2 -> 0
- net +3V3BU: track 23.5 -> 0.00 mm, vias 1 -> 0
- net NSS: track 18.2 -> 0.00 mm, vias 2 -> 0
- net +3V3ROV: track 17.4 -> 0.00 mm, vias 3 -> 0
- net +3V3BAT: track 16.7 -> 0.00 mm, vias 1 -> 0
- net CAN_STM_TX: track 15.9 -> 0.00 mm, vias 2 -> 0
- net CAN_STM_RX: track 14.7 -> 0.00 mm, vias 2 -> 0
- net SCK: track 12.2 -> 0.00 mm
- net D0: track 9.68 -> 0.00 mm
- net D1: track 9.35 -> 0.00 mm, vias 2 -> 0
- net VCC: track 8.42 -> 0.00 mm, vias 1 -> 0
- net MOSI: track 8.03 -> 0.00 mm
- net MISO: track 7.24 -> 0.00 mm
- net N$7: track 5.54 -> 0.00 mm
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- removed copper zone on layer 1, net +3V3
- removed copper zone on layer 1, net +3V3ROV
Other:
- board size 80 x 64.8 mm -> 58.4 x 64.8 mm
