File: STM_TEST/STM_TEST.sch (EAGLE design)
At the start: 25 parts, among them U1 TPS2115APWR, Y2 ECS-80-S-4X

Commit message: Routing and Stuff
Parts:
- removed LED: 100KOHM-0603-1/10W-1%, SparkFun-Resistors:100KOHM-0603-1/10W-1%
- added C3, C4: 1.0uF, SparkFun-Capacitors:1.0UF-0603-16V-10%
- added D1: (no value), SparkFun-LED:LED0603
- added J1: (no value), SparkFun-Connectors:CONN_02
- added R4: 100k, SparkFun-Resistors:100KOHM-0603-1/10W-1%
- added SW1, SW2: (no value), special:SW_DIP-2
- added U2: AZ1117EH-3.3TRG1, AZ1117EH-3.3TRG1:AZ1117EH-3.3TRG1
Connections:
- removed net N$1: R3.2, U1.D1
- new net +3V3BU: SW2.1, U1.OUT
- new net D0: R3.2, SW1.1, U1.D0
- new net D1: R4.2, SW1.2, U1.D1
- new net VCC: C3.1, J1.2, U2.IN
- net +3V3: now also SW2.3, SW2.4; no longer U1.OUT
- net +3V3ROV: now also C4.1, R4.1, SW2.2, U2.OUT
- net GND: now also C3.2, C4.2, D1.C, J1.1, SW1.3, SW1.4, U2.ADJ/GND; no longer LED.1, U1.D0
- net N$3: now also D1.A; no longer LED.2
Other:
- moved on the sheet: R3

Commit message: Board Dimensions and Connector Layout
Parts:
- added PCB1: RPI2, MicrocontrollerComponents:RPI2
- R3, R4: value 100k -> 10k
Connections:
- new net +5V: PCB1.5V@2, PCB1.5V@4
- new net CE0: PCB1.GPIO8
- new net MISO: PCB1.GPIO9
- new net MOSI: PCB1.GPIO10
- new net RESET: PCB1.GPIO4
- new net SCLK: PCB1.GPIO11
- net GND: now also PCB1.GND@14, PCB1.GND@20, PCB1.GND@25, PCB1.GND@30, PCB1.GND@34, PCB1.GND@39, PCB1.GND@6, PCB1.GND@9

Commit message: Y'all Like Samtech?
Parts:
- added R5, R6: 100k, SparkFun-Resistors:1KOHM-0603-1/10W-1%
Connections:
- net SCLK renamed SCLK_PI
- new net CAN_RX: U$2.PA11
- new net CAN_TX: U$2.PA12
- new net CS1: CR1.!_2, R5.2
- new net I2C1_SCL: U$2.PA9
- new net I2C1_SDA: U$2.PA10
- new net MISO_PI: PCB1.GPIO9
- new net MOSI_PI: PCB1.GPIO10
- new net SCK: CR1.C, R6.1, U$2.PA5
- new net SCL: PCB1.GPIO3
- new net SDA: PCB1.GPIO2
- new net UART_RXD: PCB1.GPIO15
- new net UART_TXD: PCB1.GPIO14
- net +3V3: now also R5.1
- net GND: now also R6.2
- net MISO: now also CR1.D, U$2.PA6; no longer PCB1.GPIO9
- net MOSI: now also CR1.Q, U$2.PA7; no longer PCB1.GPIO10
Changed lines of the file:
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@@
 <?xml version="1.0" encoding="utf-8"?>
 <!DOCTYPE eagle SYSTEM "eagle.dtd">
-<eagle version="9.2.0">
+<eagle version="8.6.1">
 <drawing>
 <settings>
@@
 <part name="GND22" library="supply1" library_urn="urn:adsk.eagle:library:371" deviceset="GND" device=""/>
 <part name="P+1" library="supply1" library_urn="urn:adsk.eagle:library:371" deviceset="+5V" device=""/>
+<part name="R5" library="SparkFun-Resistors" library_urn="urn:adsk.eagle:library:532" deviceset="1KOHM" device="-0603-1/10W-1%" package3d_urn="urn:adsk.eagle:package:39650/1" value="100k"/>
+<part name="+3V1" library="supply1" library_urn="urn:adsk.eagle:library:371" deviceset="+3V3" device=""/>
+<part name="R6" library="SparkFun-Resistors" library_urn="urn:adsk.eagle:library:532" deviceset="1KOHM" device="-0603-1/10W-1%" package3d_urn="urn:adsk.eagle:package:39650/1" value="100k"/>
+<part name="GND23" library="supply2" library_urn="urn:adsk.eagle:library:372" deviceset="GND" device=""/>
 </parts>
 <sheets>
@@
 <attribute name="NAME" x="333.756" y="190.5" size="1.778" layer="95" font="vector" rot="R90" align="bottom-center"/>
 <attribute name="VALUE" x="336.804" y="190.5" size="1.778" layer="96" font="vector" rot="R90" align="top-center"/>
+</instance>
+<instance part="R5" gate="G$1" x="35.56" y="223.52"/>
+<instance part="+3V1" gate="G$1" x="22.86" y="236.22">
+<attribute name="VALUE" x="20.32" y="231.14" size="1.778" layer="96" rot="R90"/>
+</instance>
+<instance part="R6" gate="G$1" x="236.22" y="180.34" rot="R180"/>
+<instance part="GND23" gate="GND" x="223.52" y="172.72">
+<attribute name="VALUE" x="221.615" y="169.545" size="1.778" layer="96"/>
 </instance>
 </instances>
@@
 <junction x="347.98" y="142.24"/>
 </segment>
+<segment>
+<pinref part="R6" gate="G$1" pin="2"/>
+<pinref part="GND23" gate="GND" pin="GND"/>
+<wire x1="231.14" y1="180.34" x2="223.52" y2="180.34" width="0.1524" layer="91"/>
+<wire x1="223.52" y1="180.34" x2="223.52" y2="175.26" width="0.1524" layer="91"/>
+</segment>
 </net>
 <net name="+3V3" class="0">
@@
 <label x="248.92" y="205.74" size="1.778" layer="95"/>
 </segment>
+<segment>
+<pinref part="R5" gate="G$1" pin="1"/>
+<wire x1="30.48" y1="223.52" x2="22.86" y2="223.52" width="0.1524" layer="91"/>
+<wire x1="22.86" y1="223.52" x2="22.86" y2="233.68" width="0.1524" layer="91"/>
+<pinref part="+3V1" gate="G$1" pin="+3V3"/>
+</segment>
 </net>
 <net name="NRST" class="0">
@@
 <wire x1="335.28" y1="185.42" x2="335.28" y2="165.1" width="0.1524" layer="91"/>
 <junction x="335.28" y="165.1"/>
+</segment>
+</net>
+<net name="MISO" class="0">
+<segment>
+<pinref part="U$2" gate="G$1" pin="PA6"/>
+<wire x1="284.48" y1="185.42" x2="284.48" y2="175.26" width="0.1524" layer="91"/>
+<label x="284.48" y="172.72" size="1.778" layer="95" rot="R90"/>
+</segment>
+<segment>
+<pinref part="CR1" gate="A" pin="D"/>
+<wire x1="114.3" y1="215.9" x2="129.54" y2="215.9" width="0.1524" layer="91"/>
+<label x="124.46" y="215.9" size="1.778" layer="95"/>
+</segment>
+</net>
+<net name="MOSI" class="0">
+<segment>
+<pinref part="U$2" gate="G$1" pin="PA7"/>
+<wire x1="289.56" y1="185.42" x2="289.56" y2="175.26" width="0.1524" layer="91"/>
+<label x="289.56" y="172.72" size="1.778" layer="95" rot="R90"/>
+</segment>
+<segment>
+<pinref part="CR1" gate="A" pin="Q"/>
+<wire x1="58.42" y1="220.98" x2="45.72" y2="220.98" width="0.1524" layer="91"/>
+<label x="45.72" y="220.98" size="1.778" layer="95"/>
+</segment>
+</net>
+<net name="CAN_TX" class="0">
+<segment>
+<pinref part="U$2" gate="G$1" pin="PA12"/>
+<wire x1="309.88" y1="213.36" x2="325.12" y2="213.36" width="0.1524" layer="91"/>
+<label x="317.5" y="213.36" size="1.778" layer="95"/>
+</segment>
+</net>
+<net name="CAN_RX" class="0">
+<segment>
+<pinref part="U$2" gate="G$1" pin="PA11"/>
+<wire x1="309.88" y1="210.82" x2="325.12" y2="210.82" width="0.1524" layer="91"/>
+<label x="317.5" y="210.82" size="1.778" layer="95"/>
+</segment>
+</net>
+<net name="I2C1_SDA" class="0">
+<segment>
+<pinref part="U$2" gate="G$1" pin="PA10"/>
+<wire x1="309.88" y1="205.74" x2="325.12" y2="205.74" width="0.1524" layer="91"/>
+<label x="317.5" y="205.74" size="1.778" layer="95"/>
+</segment>
+</net>
+<net name="I2C1_SCL" class="0">
+<segment>
+<pinref part="U$2" gate="G$1" pin="PA9"/>
+<wire x1="309.88" y1="203.2" x2="325.12" y2="203.2" width="0.1524" layer="91"/>
+<label x="317.5" y="203.2" size="1.778" layer="95"/>
+</segment>
+</net>
+<net name="SCK" class="0">
+<segment>
+<pinref part="CR1" gate="A" pin="C"/>
+<wire x1="114.3" y1="218.44" x2="129.54" y2="218.44" width="0.1524" layer="91"/>
+<label x="124.46" y="218.44" size="1.778" layer="95"/>
+</segment>
+<segment>
+<pinref part="U$2" gate="G$1" pin="PA5"/>
+<wire x1="281.94" y1="185.42" x2="281.94" y2="175.26" width="0.1524" layer="91"/>
+<label x="281.94" y="172.72" size="1.778" layer="95" rot="R90"/>
+</segment>
+<segment>
+<pinref part="R6" gate="G$1" pin="1"/>
+<wire x1="241.3" y1="180.34" x2="254" y2="180.34" width="0.1524" layer="91"/>
+<label x="248.92" y="180.34" size="1.778" layer="95"/>
+</segment>
+</net>
+<net name="CS1" class="0">
+<segment>
+<pinref part="R5" gate="G$1" pin="2"/>
+<pinref part="CR1" gate="A" pin="!_2"/>
+<wire x1="40.64" y1="223.52" x2="58.42" y2="223.52" width="0.1524" layer="91"/>
+<label x="40.64" y="223.52" size="1.778" layer="95"/>
 </segment>
 </net>
@@
 </segment>
 </net>
-<net name="SCLK" class="0">
+<net name="SCLK_PI" class="0">
 <segment>
 <pinref part="PCB1" gate="G$1" pin="GPIO11"/>
@@
 </segment>
 </net>
-<net name="MISO" class="0">
+<net name="MISO_PI" class="0">
 <segment>
 <pinref part="PCB1" gate="G$1" pin="GPIO9"/>
@@
 </segment>
 </net>
-<net name="MOSI" class="0">
+<net name="MOSI_PI" class="0">
 <segment>
 <pinref part="PCB1" gate="G$1" pin="GPIO10"/>
@@
 </segment>
 </net>
+<net name="UART_RXD" class="0">
+<segment>
+<pinref part="PCB1" gate="G$1" pin="GPIO15"/>
+<wire x1="63.5" y1="111.76" x2="45.72" y2="111.76" width="0.1524" layer="91"/>
+<label x="45.72" y="109.22" size="1.778" layer="95"/>
+</segment>
+</net>
+<net name="UART_TXD" class="0">
+<segment>
+<pinref part="PCB1" gate="G$1" pin="GPIO14"/>
+<wire x1="63.5" y1="106.68" x2="45.72" y2="106.68" width="0.1524" layer="91"/>
+<label x="45.72" y="104.14" size="1.778" layer="95"/>
+</segment>
+</net>
+<net name="SDA" class="0">
+<segment>
+<pinref part="PCB1" gate="G$1" pin="GPIO2"/>
+<wire x1="91.44" y1="96.52" x2="101.6" y2="96.52" width="0.1524" layer="91"/>
+<label x="96.52" y="96.52" size="1.778" layer="95"/>
+</segment>
+</net>
+<net name="SCL" class="0">
+<segment>
+<pinref part="PCB1" gate="G$1" pin="GPIO3"/>
+<wire x1="91.44" y1="101.6" x2="101.6" y2="101.6" width="0.1524" layer="91"/>
+<label x="96.52" y="101.6" size="1.778" layer="95"/>
+</segment>
+</net>

Commit message: Yay CAN
Parts:
- added C5, C6: 4.7nF, SparkFun-Capacitors:0.1UF-0603-25V-(+80/-20%)
- added J2: (no value), SparkFun-Connectors:CONN_02
- added R10, R11, R14, R15: 60, SparkFun-Resistors:1KOHM-0603-1/10W-1%
- added R12, R13, R16, R17: 0, SparkFun-Resistors:1KOHM-0603-1/10W-1%
Connections:
- removed net CS1: CR1.!_2, R5.2
- new net CAN_H: J2.2, R12.2, R16.2
- new net CAN_L: J2.1, R13.2, R17.2
- new net N$1: C5.2, R10.1, R11.2
- new net N$10: R14.2, R16.1
- new net N$4: R11.1, R13.1
- new net N$5: R10.2, R12.1
- new net N$8: C6.2, R14.1, R15.2
- new net N$9: R15.1, R17.1
- new net NSS: CR1.!_2, R5.2, U$2.PA4
- net GND: now also C5.1, C6.1
Other:
- note added: "CAN TERMINATION"
- note added: "Connect CAN nodes between these two terminators if can bus only being used on this board. (bridge zero ohm resistors)"
Changed lines of the file:
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@@
 <part name="R6" library="SparkFun-Resistors" library_urn="urn:adsk.eagle:library:532" deviceset="1KOHM" device="-0603-1/10W-1%" package3d_urn="urn:adsk.eagle:package:39650/1" value="100k"/>
 <part name="GND23" library="supply2" library_urn="urn:adsk.eagle:library:372" deviceset="GND" device=""/>
+<part name="J2" library="SparkFun-Connectors" deviceset="CONN_02" device=""/>
+<part name="R10" library="SparkFun-Resistors" library_urn="urn:adsk.eagle:library:532" deviceset="1KOHM" device="-0603-1/10W-1%" package3d_urn="urn:adsk.eagle:package:39650/1" value="60"/>
+<part name="R11" library="SparkFun-Resistors" library_urn="urn:adsk.eagle:library:532" deviceset="1KOHM" device="-0603-1/10W-1%" package3d_urn="urn:adsk.eagle:package:39650/1" value="60"/>
+<part name="C5" library="SparkFun-Capacitors" library_urn="urn:adsk.eagle:library:510" deviceset="0.1UF" device="-0603-25V-(+80/-20%)" package3d_urn="urn:adsk.eagle:package:37414/1" value="4.7nF"/>
+<part name="GND24" library="supply1" library_urn="urn:adsk.eagle:library:371" deviceset="GND" device=""/>
+<part name="R12" library="SparkFun-Resistors" library_urn="urn:adsk.eagle:library:532" deviceset="1KOHM" device="-0603-1/10W-1%" package3d_urn="urn:adsk.eagle:package:39650/1" value="0"/>
+<part name="R13" library="SparkFun-Resistors" library_urn="urn:adsk.eagle:library:532" deviceset="1KOHM" device="-0603-1/10W-1%" package3d_urn="urn:adsk.eagle:package:39650/1" value="0"/>
+<part name="R14" library="SparkFun-Resistors" library_urn="urn:adsk.eagle:library:532" deviceset="1KOHM" device="-0603-1/10W-1%" package3d_urn="urn:adsk.eagle:package:39650/1" value="60"/>
+<part name="R15" library="SparkFun-Resistors" library_urn="urn:adsk.eagle:library:532" deviceset="1KOHM" device="-0603-1/10W-1%" package3d_urn="urn:adsk.eagle:package:39650/1" value="60"/>
+<part name="C6" library="SparkFun-Capacitors" library_urn="urn:adsk.eagle:library:510" deviceset="0.1UF" device="-0603-25V-(+80/-20%)" package3d_urn="urn:adsk.eagle:package:37414/1" value="4.7nF"/>
+<part name="GND25" library="supply1" library_urn="urn:adsk.eagle:library:371" deviceset="GND" device=""/>
+<part name="R16" library="SparkFun-Resistors" library_urn="urn:adsk.eagle:library:532" deviceset="1KOHM" device="-0603-1/10W-1%" package3d_urn="urn:adsk.eagle:package:39650/1" value="0"/>
+<part name="R17" library="SparkFun-Resistors" library_urn="urn:adsk.eagle:library:532" deviceset="1KOHM" device="-0603-1/10W-1%" package3d_urn="urn:adsk.eagle:package:39650/1" value="0"/>
 </parts>
 <sheets>
@@
 <text x="246.38" y="132.08" size="1.778" layer="91">Pin 17 (VDDIO2)</text>
 <text x="274.32" y="132.08" size="1.778" layer="91">Pin 5 (VDDA)</text>
+<text x="86.36" y="144.78" size="1.778" layer="91">CAN TERMINATION</text>
+<text x="76.2" y="119.38" size="1.778" layer="91">Connect CAN nodes between these two
+ terminators if can bus only being used on this
+ board. (bridge zero ohm resistors)</text>
 </plain>
 <instances>
@@
 <attribute name="VALUE" x="221.615" y="169.545" size="1.778" layer="96"/>
 </instance>
+<instance part="J2" gate="G$1" x="20.32" y="175.26">
+<attribute name="VALUE" x="17.78" y="170.434" size="1.778" layer="96" font="vector"/>
+<attribute name="NAME" x="17.78" y="180.848" size="1.778" layer="95" font="vector"/>
+</instance>
+<instance part="R10" gate="G$1" x="53.34" y="129.54" rot="R90"/>
+<instance part="R11" gate="G$1" x="53.34" y="114.3" rot="R90"/>
+<instance part="C5" gate="G$1" x="35.56" y="119.38" rot="R180"/>
+<instance part="GND24" gate="1" x="35.56" y="99.06">
+<attribute name="VALUE" x="33.02" y="96.52" size="1.778" layer="96"/>
+</instance>
+<instance part="R12" gate="G$1" x="68.58" y="137.16"/>
+<instance part="R13" gate="G$1" x="68.58" y="106.68"/>
+<instance part="R14" gate="G$1" x="142.24" y="129.54" rot="MR90"/>
+<instance part="R15" gate="G$1" x="142.24" y="114.3" rot="MR90"/>
+<instance part="C6" gate="G$1" x="160.02" y="119.38" rot="MR180"/>
+<instance part="GND25" gate="1" x="160.02" y="99.06" rot="MR0">
+<attribute name="VALUE" x="162.56" y="96.52" size="1.778" layer="96" rot="MR0"/>
+</instance>
+<instance part="R16" gate="G$1" x="127" y="137.16" rot="MR0"/>
+<instance part="R17" gate="G$1" x="127" y="106.68" rot="MR0"/>
 </instances>
 <busses>
@@
 <wire x1="223.52" y1="180.34" x2="223.52" y2="175.26" width="0.1524" layer="91"/>
 </segment>
+<segment>
+<pinref part="GND24" gate="1" pin="GND"/>
+<pinref part="C5" gate="G$1" pin="1"/>
+<wire x1="35.56" y1="101.6" x2="35.56" y2="114.3" width="0.1524" layer="91"/>
+</segment>
+<segment>
+<pinref part="GND25" gate="1" pin="GND"/>
+<pinref part="C6" gate="G$1" pin="1"/>
+<wire x1="160.02" y1="101.6" x2="160.02" y2="114.3" width="0.1524" layer="91"/>
+</segment>
 </net>
 <net name="+3V3" class="0">
@@
 </segment>
 </net>
-<net name="CS1" class="0">
+<net name="NSS" class="0">
 <segment>
 <pinref part="R5" gate="G$1" pin="2"/>
@@
 <label x="40.64" y="223.52" size="1.778" layer="95"/>
 </segment>
-</net>
+<segment>
+<pinref part="U$2" gate="G$1" pin="PA4"/>
+<wire x1="279.4" y1="185.42" x2="279.4" y2="172.72" width="0.1524" layer="91"/>
+<label x="279.4" y="172.72" size="1.778" layer="95" rot="R90"/>
+</segment>
+</net>
+<net name="CAN_H" class="0">
+<segment>
+<pinref part="J2" gate="G$1" pin="2"/>
+<wire x1="27.94" y1="177.8" x2="43.18" y2="177.8" width="0.1524" layer="91"/>
+<label x="35.56" y="177.8" size="1.778" layer="95"/>
+</segment>
+<segment>
+<pinref part="R12" gate="G$1" pin="2"/>
+<wire x1="73.66" y1="137.16" x2="86.36" y2="137.16" width="0.1524" layer="91"/>
+<label x="78.74" y="137.16" size="1.778" layer="95"/>
+</segment>
+<segment>
+<pinref part="R16" gate="G$1" pin="2"/>
+<wire x1="121.92" y1="137.16" x2="109.22" y2="137.16" width="0.1524" layer="91"/>
+<label x="116.84" y="137.16" size="1.778" layer="95" rot="MR0"/>
+</segment>
+</net>
+<net name="CAN_L" class="0">
+<segment>
+<pinref part="J2" gate="G$1" pin="1"/>
+<wire x1="27.94" y1="175.26" x2="43.18" y2="175.26" width="0.1524" layer="91"/>
+<label x="35.56" y="175.26" size="1.778" layer="95"/>
+</segment>
+<segment>
+<pinref part="R13" gate="G$1" pin="2"/>
+<wire x1="73.66" y1="106.68" x2="86.36" y2="106.68" width="0.1524" layer="91"/>
+<label x="78.74" y="106.68" size="1.778" layer="95"/>
+</segment>
+<segment>
+<pinref part="R17" gate="G$1" pin="2"/>
+<wire x1="121.92" y1="106.68" x2="109.22" y2="106.68" width="0.1524" layer="91"/>
+<label x="116.84" y="106.68" size="1.778" layer="95" rot="MR0"/>
+</segment>
+</net>
+<net name="N$1" class="0">
+<segment>
+<pinref part="R10" gate="G$1" pin="1"/>
+<pinref part="R11" gate="G$1" pin="2"/>
+<wire x1="53.34" y1="124.46" x2="53.34" y2="121.92" width="0.1524" layer="91"/>
+<pinref part="C5" gate="G$1" pin="2"/>
+<wire x1="53.34" y1="121.92" x2="53.34" y2="119.38" width="0.1524" layer="91"/>
+<wire x1="35.56" y1="121.92" x2="53.34" y2="121.92" width="0.1524" layer="91"/>
+<junction x="53.34" y="121.92"/>
+</segment>
+</net>
+<net name="N$4" class="0">
+<segment>
+<pinref part="R11" gate="G$1" pin="1"/>
+<pinref part="R13" gate="G$1" pin="1"/>
+<wire x1="53.34" y1="109.22" x2="53.34" y2="106.68" width="0.1524" layer="91"/>
+<wire x1="53.34" y1="106.68" x2="63.5" y2="106.68" width="0.1524" layer="91"/>
+</segment>
+</net>
+<net name="N$5" class="0">
+<segment>
+<pinref part="R10" gate="G$1" pin="2"/>
+<pinref part="R12" gate="G$1" pin="1"/>
+<wire x1="53.34" y1="134.62" x2="53.34" y2="137.16" width="0.1524" layer="91"/>
+<wire x1="53.34" y1="137.16" x2="63.5" y2="137.16" width="0.1524" layer="91"/>
+</segment>
+</net>
+<net name="N$8" class="0">
+<segment>
+<pinref part="R14" gate="G$1" pin="1"/>
+<pinref part="R15" gate="G$1" pin="2"/>
+<wire x1="142.24" y1="124.46" x2="142.24" y2="121.92" width="0.1524" layer="91"/>
+<pinref part="C6" gate="G$1" pin="2"/>
+<wire x1="142.24" y1="121.92" x2="142.24" y2="119.38" width="0.1524" layer="91"/>
+<wire x1="160.02" y1="121.92" x2="142.24" y2="121.92" width="0.1524" layer="91"/>
+<junction x="142.24" y="121.92"/>
+</segment>
+</net>
+<net name="N$9" class="0">
+<segment>
+<pinref part="R15" gate="G$1" pin="1"/>
+<pinref part="R17" gate="G$1" pin="1"/>
+<wire x1="142.24" y1="109.22" x2="142.24" y2="106.68" width="0.1524" layer="91"/>
+<wire x1="142.24" y1="106.68" x2="132.08" y2="106.68" width="0.1524" layer="91"/>
+</segment>
+</net>
+<net name="N$10" class="0">
+<segment>
+<pinref part="R14" gate="G$1" pin="2"/>
+<pinref part="R16" gate="G$1" pin="1"/>
+<wire x1="142.24" y1="134.62" x2="142.24" y2="137.16" width="0.1524" layer="91"/>
+<wire x1="142.24" y1="137.16" x2="132.08" y2="137.16" width="0.1524" layer="91"/>
+</segment>
+</net>
