File: STM_TEST/STM_TEST.sch (EAGLE design)
At the start: 46 parts, among them U1 TPS2115APWR, U2 AZ1117EH-3.3TRG1, Y2 ECS-80-S-4X

Commit message: Board Layout
Parts:
- added C7: 100nF, SparkFun-Capacitors:4.7UF0603
- added U$1: TCAN337D, PI_Shield_Library:TCAN337D
Connections:
- removed net CAN_RX: U$2.PA11
- removed net CAN_TX: U$2.PA12
- new net CAN_STM_RX: U$1.TXD, U$2.PA11
- new net CAN_STM_TX: U$1.RXD, U$2.PA12
- net +3V3: now also C7.1, U$1.VCC
- net CAN_H: now also U$1.CANH
- net CAN_L: now also U$1.CANL
- net GND: now also C7.2, U$1.GND
Other:
- note added: "EEPROM"
- moved on the sheet: J2
Changed lines of the file:
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@@
 <part name="R16" library="SparkFun-Resistors" library_urn="urn:adsk.eagle:library:532" deviceset="1KOHM" device="-0603-1/10W-1%" package3d_urn="urn:adsk.eagle:package:39650/1" value="0"/>
 <part name="R17" library="SparkFun-Resistors" library_urn="urn:adsk.eagle:library:532" deviceset="1KOHM" device="-0603-1/10W-1%" package3d_urn="urn:adsk.eagle:package:39650/1" value="0"/>
+<part name="U$1" library="PI_Shield_Library" deviceset="TCAN337D" device=""/>
+<part name="C7" library="SparkFun-Capacitors" library_urn="urn:adsk.eagle:library:510" deviceset="4.7UF" device="0603" package3d_urn="urn:adsk.eagle:package:37414/1" value="100nF"/>
+<part name="+3V2" library="supply1" library_urn="urn:adsk.eagle:library:371" deviceset="+3V3" device=""/>
+<part name="GND26" library="supply1" library_urn="urn:adsk.eagle:library:371" deviceset="GND" device=""/>
+<part name="GND27" library="supply1" library_urn="urn:adsk.eagle:library:371" deviceset="GND" device=""/>
 </parts>
 <sheets>
@@
  terminators if can bus only being used on this
  board. (bridge zero ohm resistors)</text>
+<text x="81.28" y="238.76" size="1.778" layer="91">EEPROM</text>
 </plain>
 <instances>
@@
 <attribute name="VALUE" x="221.615" y="169.545" size="1.778" layer="96"/>
 </instance>
-<instance part="J2" gate="G$1" x="20.32" y="175.26">
-<attribute name="VALUE" x="17.78" y="170.434" size="1.778" layer="96" font="vector"/>
-<attribute name="NAME" x="17.78" y="180.848" size="1.778" layer="95" font="vector"/>
+<instance part="J2" gate="G$1" x="91.44" y="83.82">
+<attribute name="VALUE" x="88.9" y="78.994" size="1.778" layer="96" font="vector"/>
+<attribute name="NAME" x="88.9" y="89.408" size="1.778" layer="95" font="vector"/>
 </instance>
 <instance part="R10" gate="G$1" x="53.34" y="129.54" rot="R90"/>
@@
 <instance part="R16" gate="G$1" x="127" y="137.16" rot="MR0"/>
 <instance part="R17" gate="G$1" x="127" y="106.68" rot="MR0"/>
+<instance part="U$1" gate="G$1" x="99.06" y="50.8"/>
+<instance part="C7" gate="G$1" x="45.72" y="50.8">
+<attribute name="NAME" x="47.244" y="53.721" size="1.778" layer="95" font="vector"/>
+<attribute name="VALUE" x="47.244" y="48.641" size="1.778" layer="96" font="vector"/>
+</instance>
+<instance part="+3V2" gate="G$1" x="45.72" y="71.12">
+<attribute name="VALUE" x="43.18" y="66.04" size="1.778" layer="96" rot="R90"/>
+</instance>
+<instance part="GND26" gate="1" x="45.72" y="40.64">
+<attribute name="VALUE" x="43.18" y="38.1" size="1.778" layer="96"/>
+</instance>
+<instance part="GND27" gate="1" x="81.28" y="33.02">
+<attribute name="VALUE" x="78.74" y="30.48" size="1.778" layer="96"/>
+</instance>
 </instances>
 <busses>
@@
 <wire x1="160.02" y1="101.6" x2="160.02" y2="114.3" width="0.1524" layer="91"/>
 </segment>
+<segment>
+<pinref part="C7" gate="G$1" pin="2"/>
+<pinref part="GND26" gate="1" pin="GND"/>
+<wire x1="45.72" y1="48.26" x2="45.72" y2="43.18" width="0.1524" layer="91"/>
+</segment>
+<segment>
+<pinref part="U$1" gate="G$1" pin="GND"/>
+<pinref part="GND27" gate="1" pin="GND"/>
+<wire x1="83.82" y1="43.18" x2="81.28" y2="43.18" width="0.1524" layer="91"/>
+<wire x1="81.28" y1="43.18" x2="81.28" y2="35.56" width="0.1524" layer="91"/>
+</segment>
 </net>
 <net name="+3V3" class="0">
@@
 <pinref part="+3V1" gate="G$1" pin="+3V3"/>
 </segment>
+<segment>
+<pinref part="+3V2" gate="G$1" pin="+3V3"/>
+<wire x1="45.72" y1="55.88" x2="45.72" y2="58.42" width="0.1524" layer="91"/>
+<pinref part="C7" gate="G$1" pin="1"/>
+<pinref part="U$1" gate="G$1" pin="VCC"/>
+<wire x1="45.72" y1="58.42" x2="45.72" y2="68.58" width="0.1524" layer="91"/>
+<wire x1="83.82" y1="58.42" x2="45.72" y2="58.42" width="0.1524" layer="91"/>
+<junction x="45.72" y="58.42"/>
+</segment>
 </net>
 <net name="NRST" class="0">
@@
 </segment>
 </net>
-<net name="CAN_TX" class="0">
+<net name="CAN_STM_TX" class="0">
 <segment>
 <pinref part="U$2" gate="G$1" pin="PA12"/>
@@
 <label x="317.5" y="213.36" size="1.778" layer="95"/>
 </segment>
-</net>
-<net name="CAN_RX" class="0">
+<segment>
+<pinref part="U$1" gate="G$1" pin="RXD"/>
+<wire x1="83.82" y1="48.26" x2="66.04" y2="48.26" width="0.1524" layer="91"/>
+<label x="60.96" y="48.26" size="1.778" layer="95"/>
+</segment>
+</net>
+<net name="CAN_STM_RX" class="0">
 <segment>
 <pinref part="U$2" gate="G$1" pin="PA11"/>
 <wire x1="309.88" y1="210.82" x2="325.12" y2="210.82" width="0.1524" layer="91"/>
 <label x="317.5" y="210.82" size="1.778" layer="95"/>
+</segment>
+<segment>
+<pinref part="U$1" gate="G$1" pin="TXD"/>
+<wire x1="83.82" y1="53.34" x2="66.04" y2="53.34" width="0.1524" layer="91"/>
+<label x="60.96" y="53.34" size="1.778" layer="95"/>
 </segment>
 </net>
@@
 <segment>
 <pinref part="J2" gate="G$1" pin="2"/>
-<wire x1="27.94" y1="177.8" x2="43.18" y2="177.8" width="0.1524" layer="91"/>
-<label x="35.56" y="177.8" size="1.778" layer="95"/>
+<wire x1="99.06" y1="86.36" x2="114.3" y2="86.36" width="0.1524" layer="91"/>
+<label x="106.68" y="86.36" size="1.778" layer="95"/>
 </segment>
 <segment>
@@
 <label x="116.84" y="137.16" size="1.778" layer="95" rot="MR0"/>
 </segment>
+<segment>
+<pinref part="U$1" gate="G$1" pin="CANH"/>
+<wire x1="114.3" y1="53.34" x2="132.08" y2="53.34" width="0.1524" layer="91"/>
+<label x="124.46" y="53.34" size="1.778" layer="95"/>
+</segment>
 </net>
 <net name="CAN_L" class="0">
 <segment>
 <pinref part="J2" gate="G$1" pin="1"/>
-<wire x1="27.94" y1="175.26" x2="43.18" y2="175.26" width="0.1524" layer="91"/>
-<label x="35.56" y="175.26" size="1.778" layer="95"/>
+<wire x1="99.06" y1="83.82" x2="114.3" y2="83.82" width="0.1524" layer="91"/>
+<label x="106.68" y="83.82" size="1.778" layer="95"/>
 </segment>
 <segment>
@@
 <label x="116.84" y="106.68" size="1.778" layer="95" rot="MR0"/>
 </segment>
-</net>
+<segment>
+<pinref part="U$1" gate="G$1" pin="CANL"/>
+<wire x1="114.3" y1="48.26" x2="132.08" y2="48.26" width="0.1524" layer="91"/>
+<label x="124.46" y="48.26" size="1.778" layer="95"/>
+</segment>
+</net>

Commit message: things
Parts:
- removed R12, R13, R16, R17: 0, SparkFun-Resistors:1KOHM-0603-1/10W-1%
- removed R14, R15: 60, SparkFun-Resistors:1KOHM-0603-1/10W-1%
- added U$3: TCAN337D, PI_Shield_Library:TCAN337D
- added U$5: MCP2515, PI_Shield_Library:MCP2515
- C6: value 4.7nF -> 100nF; device SparkFun-Capacitors:0.1UF-0603-25V-(+80/-20%) -> SparkFun-Capacitors:4.7UF0603
Connections:
- removed net N$4: R11.1, R13.1
- removed net N$5: R10.2, R12.1
- new net CAN_PI_RX: U$3.TXD, U$5.RXCAN
- new net CAN_PI_TX: U$3.RXD, U$5.TXCAN
- new net N$11: U$5.CS
- net +3V3: now also C6.1, U$3.VCC
- net CAN_H: now also R10.2, U$3.CANH; no longer R12.2, R16.2
- net CAN_L: now also R11.1, U$3.CANL; no longer R13.2, R17.2
- net GND: now also C6.2, U$3.GND; no longer C6.1
- net N$10: now also U$5.SO; no longer R14.2, R16.1
- net N$8: now also U$5.SCK; no longer C6.2, R14.1, R15.2
- net N$9: now also U$5.SI; no longer R15.1, R17.1
Other:
- note removed: "Connect CAN nodes between these two terminators if can bus only being used on this board. (bridge zero ohm resistors)"

Commit message: reroute
Parts:
- added C10, C8, C9: 100nF, SparkFun-Capacitors:4.7UF0603
- added C11: 18pF, SparkFun-Capacitors:4.7UF0603
- added Y1: ECS-80-S-4X, ECS-80-S-4X:ECS-80-S-4X
- C18: value 100nF -> 18pF
Connections:
- removed net N$10: U$5.SO
- removed net N$11: U$5.CS
- removed net N$8: U$5.SCK
- removed net N$9: U$5.SI
- new net OSC1: C18.1, U$5.OSC1, Y1.2
- new net OSC2: C11.1, U$5.OSC2, Y1.1
- net +3V3: now also C8.1, C9.1, U$5.VDD
- net +3V3BU: now also SW2.2; no longer SW2.1
- net +3V3ROV: now also SW2.1; no longer SW2.2
- net CE0: now also U$5.CS
- net D0: now also R4.2, SW1.2; no longer R3.2, SW1.1
- net D1: now also R3.2, SW1.1; no longer R4.2, SW1.2
- net GND: now also C10.2, C11.2, C8.2, C9.2, U$5.VSS
- net MISO_PI: now also U$5.SO
- net MOSI_PI: now also U$5.SI
- net NRST: now also C10.1; no longer C18.1
- net SCLK_PI: now also U$5.SCK
