File: PI_Shield.brd (EAGLE design)
At the start: 80.1 x 86.7 mm, 59 parts, among them Q1 220mA/50V/3.5Ω, Q3 220mA/50V/3.5Ω, Q4 220mA/50V/3.5Ω, Q5 2.5A/30V/105mΩ, U1 MAX1136EUA-T, U2 AZ1117EH-3.3TRG1, Y1 ECS-80-S-4X

Commit message: Minor Changes to Pi Shield
Parts:
- added R20: 4.7k, SparkFun-Resistors:0603
- added U$12: DF13-3P-1.25DSA, con-hirose-df13:DF13-3P-1.25DSA
- moved U$11 6.98 mm to (4.91, 35.2)
- moved U$4 5.71 mm to (4.92, 26.5)
- moved R6 4.08 mm to (69.9, 16.1)
- moved Q4 2.93 mm to (63.2, 20.5), turned to 270 degrees
- moved R7 2.82 mm to (66.3, 16.1)
- moved R4 2.67 mm to (63.0, 26.0)
- moved U$6 2.16 mm to (4.92, 17.2)
- moved C5 2.12 mm to (65.3, 43.8), turned to 270 degrees
- moved D1 1.58 mm to (57.1, 40.4), turned to 90 degrees
- moved R3 1.40 mm to (71.4, 34.9)
- moved R1 1.03 mm to (40.6, 39.6), turned to 0 degrees
- moved R5 0.89 mm to (69.0, 25.0)
- moved Q5 0.52 mm to (45.1, 34.8)
- moved C6 0.52 mm to (62.2, 16.0)
- moved R16 0.51 mm to (40.3, 35.0)
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Connections:
- new net PWM: PCB1.P$32, U$12.P$2
- net 5V: now also R20.2, U$12.P$1
- net DI: now also PCB1.P$40, R20.1; no longer PCB1.P$36
- net GND: now also U$12.P$3
Routing:
- net 3V3: track 451.4 -> 385.9 mm
- net SDA: track 86.7 -> 109.5 mm
- net 5V: track 223.5 -> 203.3 mm
- net IMU_INT: track 49.8 -> 34.8 mm, vias 2 -> 1
- net PWM: track 0.00 -> 13.1 mm
- net RESET: track 20.7 -> 8.73 mm
- net CANL: track 58.1 -> 48.9 mm, vias 3 -> 0
- net CANH: track 57.7 -> 48.8 mm
- net TXCAN: track 29.3 -> 21.3 mm
- net AMP_FAULT: track 22.4 -> 14.7 mm
- net IMU_RESET: track 52.2 -> 44.6 mm
- net CLK: track 50.0 -> 57.4 mm
- net DI: track 9.99 -> 16.8 mm, vias 0 -> 1
- net MISO: track 51.8 -> 57.4 mm
- net AIN: track 41.3 -> 36.0 mm
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- removed copper zone on layer 16, net SCL
- removed copper zone on layer 1, net SDA

Commit message: Added Connectors, need to route
Parts:
- added J1, J2: (no value), SparkFun-Connectors:1X04
- added J6, J7: (no value), SparkFun-Connectors:1X02
- added U$13, U$14: T2I, BackplaneParts:T2I
- R1: value 10k -> 1k
- R10: value 47 -> 1k
- R2: value 1k -> 10k
- moved R20 61.8 mm to (68.0, 39.0), turned to 0 degrees
- moved U$9 60.0 mm to (62.7, 36.5), turned to 0 degrees
- moved U$12 57.7 mm to (62.7, 43.8), turned to 0 degrees
- moved C5 28.9 mm to (49.4, 19.7), flipped to the bottom, turned to 90 degrees
- moved D2 24.6 mm to (45.5, 14.1), flipped to the bottom
- moved R5 24.1 mm to (45.5, 19.7), flipped to the bottom
- moved R4 22.9 mm to (41.0, 19.7), flipped to the bottom, turned to 90 degrees
- moved Q4 22.2 mm to (42.0, 14.4), flipped to the bottom, turned to 180 degrees
- moved U$2 20.2 mm to (54.5, 21.8), flipped to the bottom, turned to 180 degrees
- moved R3 17.0 mm to (57.5, 25.1), flipped to the bottom, turned to 0 degrees
- moved R10 15.9 mm to (37.5, 39.1)
- moved J5 13.7 mm to (74.9, 59.8)
- moved D1 9.31 mm to (47.8, 41.3), turned to 270 degrees
- moved U$10 5.66 mm to (77.7, 17.8)
- moved D4 5.31 mm to (50.6, 38.2), turned to 0 degrees
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Connections:
- removed net N$6: D1.A, R10.2
- new net AIN2: J2.2, U1.3
- new net DI1: PCB1.P$36, U$14.3
- new net DI2: PCB1.P$38, U$14.2
- new net DI3: PCB1.P$40, U$14.1
- new net RESET_TO_PI: R10.2
- net 3V3: now also J1.4, J2.3, J6.2, J7.2
- net 5V: now also J2.4
- net CANH: now also U$13.2
- net CANL: now also U$13.3
- net DI: no longer PCB1.P$40
- net GND: now also J1.1, J2.1, J6.1, J7.1, U$14.4
- net N$3: now also D1.A
- net SCL: now also J1.2
- net SDA: now also J1.3
Routing:
- net SDA: track 109.5 -> 137.1 mm
- net SCL: track 109.5 -> 133.8 mm
- net IMU_RESET: track 44.6 -> 25.0 mm, vias 2 -> 1
- net TXCAN: track 21.3 -> 40.5 mm, vias 2 -> 1
- net 5V: track 203.3 -> 220.1 mm
- net PWM: track 13.1 -> 0.00 mm
- net CANH: track 48.8 -> 61.3 mm, vias 2 -> 4
- net DI3: track 0.00 -> 12.1 mm
- net DI2: track 0.00 -> 11.9 mm
- net DI1: track 0.00 -> 11.6 mm
- net FAULT: track 13.6 -> 24.7 mm
- net DI: track 16.8 -> 6.43 mm, vias 1 -> 0
- net RXCAN: track 21.1 -> 26.4 mm, vias 2 -> 1
- net N$1: track 3.83 -> 8.55 mm, vias 0 -> 2
- net 3V3: track 385.9 -> 389.7 mm, vias 0 -> 2
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