File: PI_Shield.sch (EAGLE design)
At the start: 59 parts, among them Q1 220mA/50V/3.5Ω, Q3 220mA/50V/3.5Ω, Q4 220mA/50V/3.5Ω, Q5 2.5A/30V/105mΩ, U1 MAX1136EUA-T, U2 AZ1117EH-3.3TRG1, Y1 ECS-80-S-4X

Commit message: Almost Done
Connections:
- removed net IMU_NET: PCB1.GPIO6
- new net OSC1_XTAL: C2.2, R19.1, Y1.1
- new net OSC2_XTAL: C1.2, R11.1, Y1.2
- net CLK: now also J4.2; no longer J4.3
- net CS: now also J4.5; no longer J4.2
- net DI: now also PCB1.GPIO16; no longer PCB1.GPIO23
- net IMU_INT: now also PCB1.GPIO22
- net IMU_RESET: now also PCB1.GPIO27; no longer PCB1.GPIO13
- net MOSI: now also J4.3; no longer J4.5
- net OSC1: no longer C2.2, R19.1, Y1.1
- net OSC2: no longer C1.2, R11.1, Y1.2
Changed lines of the file:
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@@
-</segment>
-<segment>
-<wire x1="35.56" y1="55.88" x2="43.18" y2="55.88" width="0.1524" layer="91"/>
-<pinref part="C2" gate="G$1" pin="2"/>
-<pinref part="Y1" gate="G$1" pin="1"/>
-<wire x1="43.18" y1="58.42" x2="43.18" y2="55.88" width="0.1524" layer="91"/>
-<pinref part="R19" gate="G$1" pin="1"/>
-<wire x1="43.18" y1="55.88" x2="50.8" y2="55.88" width="0.1524" layer="91"/>
-<junction x="43.18" y="55.88"/>
 </segment>
 <segment>
@@
 <wire x1="40.64" y1="127" x2="27.94" y2="127" width="0.1524" layer="91"/>
 <label x="27.94" y="127" size="1.778" layer="95"/>
-</segment>
-<segment>
-<pinref part="Y1" gate="G$1" pin="2"/>
-<wire x1="43.18" y1="68.58" x2="43.18" y2="71.12" width="0.1524" layer="91"/>
-<pinref part="C1" gate="G$1" pin="2"/>
-<wire x1="35.56" y1="71.12" x2="43.18" y2="71.12" width="0.1524" layer="91"/>
-<junction x="43.18" y="71.12"/>
-<pinref part="R11" gate="G$1" pin="1"/>
-<wire x1="43.18" y1="71.12" x2="50.8" y2="71.12" width="0.1524" layer="91"/>
 </segment>
 <segment>
@@
 <wire x1="129.54" y1="71.12" x2="129.54" y2="73.66" width="0.1524" layer="91"/>
 <pinref part="D1" gate="G$1" pin="A"/>
+</segment>
+</net>
+<net name="OSC2_XTAL" class="0">
+<segment>
+<pinref part="C1" gate="G$1" pin="2"/>
+<pinref part="R11" gate="G$1" pin="1"/>
+<wire x1="35.56" y1="71.12" x2="43.18" y2="71.12" width="0.1524" layer="91"/>
+<pinref part="Y1" gate="G$1" pin="2"/>
+<wire x1="43.18" y1="71.12" x2="50.8" y2="71.12" width="0.1524" layer="91"/>
+<wire x1="43.18" y1="68.58" x2="43.18" y2="71.12" width="0.1524" layer="91"/>
+<junction x="43.18" y="71.12"/>
+<label x="38.1" y="76.2" size="1.778" layer="95"/>
+</segment>
+</net>
+<net name="OSC1_XTAL" class="0">
+<segment>
+<pinref part="C2" gate="G$1" pin="2"/>
+<pinref part="R19" gate="G$1" pin="1"/>
+<wire x1="35.56" y1="55.88" x2="43.18" y2="55.88" width="0.1524" layer="91"/>
+<pinref part="Y1" gate="G$1" pin="1"/>
+<wire x1="43.18" y1="55.88" x2="50.8" y2="55.88" width="0.1524" layer="91"/>
+<wire x1="43.18" y1="58.42" x2="43.18" y2="55.88" width="0.1524" layer="91"/>
+<junction x="43.18" y="55.88"/>
+<label x="38.1" y="53.34" size="1.778" layer="95"/>
 </segment>
 </net>
@@
 <net name="MOSI" class="0">
 <segment>
+<pinref part="PCB1" gate="G$1" pin="GPIO10"/>
+<wire x1="45.72" y1="66.04" x2="55.88" y2="66.04" width="0.1524" layer="91"/>
+<label x="50.8" y="66.04" size="1.778" layer="95"/>
+</segment>
+<segment>
+<pinref part="J4" gate="G$1" pin="3"/>
+<wire x1="208.28" y1="38.1" x2="220.98" y2="38.1" width="0.1524" layer="91"/>
+<label x="213.36" y="38.1" size="1.778" layer="95"/>
+</segment>
+</net>
+<net name="MISO" class="0">
+<segment>
+<pinref part="J4" gate="G$1" pin="4"/>
+<wire x1="208.28" y1="40.64" x2="220.98" y2="40.64" width="0.1524" layer="91"/>
+<label x="213.36" y="40.64" size="1.778" layer="95"/>
+</segment>
+<segment>
+<pinref part="PCB1" gate="G$1" pin="GPIO9"/>
+<wire x1="45.72" y1="71.12" x2="55.88" y2="71.12" width="0.1524" layer="91"/>
+<label x="50.8" y="71.12" size="1.778" layer="95"/>
+</segment>
+</net>
+<net name="CLK" class="0">
+<segment>
+<pinref part="PCB1" gate="G$1" pin="GPIO11"/>
+<wire x1="45.72" y1="76.2" x2="55.88" y2="76.2" width="0.1524" layer="91"/>
+<label x="50.8" y="76.2" size="1.778" layer="95"/>
+</segment>
+<segment>
+<pinref part="J4" gate="G$1" pin="2"/>
+<wire x1="208.28" y1="35.56" x2="220.98" y2="35.56" width="0.1524" layer="91"/>
+<label x="213.36" y="35.56" size="1.778" layer="95"/>
+</segment>
+</net>
+<net name="CS" class="0">
+<segment>
+<pinref part="PCB1" gate="G$1" pin="GPIO8"/>
+<wire x1="17.78" y1="76.2" x2="7.62" y2="76.2" width="0.1524" layer="91"/>
+<label x="7.62" y="76.2" size="1.778" layer="95"/>
+</segment>
+<segment>
 <pinref part="J4" gate="G$1" pin="5"/>
 <wire x1="208.28" y1="43.18" x2="220.98" y2="43.18" width="0.1524" layer="91"/>
 <label x="213.36" y="43.18" size="1.778" layer="95"/>
-</segment>
-<segment>
-<pinref part="PCB1" gate="G$1" pin="GPIO10"/>
-<wire x1="45.72" y1="66.04" x2="55.88" y2="66.04" width="0.1524" layer="91"/>
-<label x="50.8" y="66.04" size="1.778" layer="95"/>
-</segment>
-</net>
-<net name="MISO" class="0">
-<segment>
-<pinref part="J4" gate="G$1" pin="4"/>
-<wire x1="208.28" y1="40.64" x2="220.98" y2="40.64" width="0.1524" layer="91"/>
-<label x="213.36" y="40.64" size="1.778" layer="95"/>
-</segment>
-<segment>
-<pinref part="PCB1" gate="G$1" pin="GPIO9"/>
-<wire x1="45.72" y1="71.12" x2="55.88" y2="71.12" width="0.1524" layer="91"/>
-<label x="50.8" y="71.12" size="1.778" layer="95"/>
-</segment>
-</net>
-<net name="CLK" class="0">
-<segment>
-<pinref part="J4" gate="G$1" pin="3"/>
-<wire x1="208.28" y1="38.1" x2="220.98" y2="38.1" width="0.1524" layer="91"/>
-<label x="213.36" y="38.1" size="1.778" layer="95"/>
-</segment>
-<segment>
-<pinref part="PCB1" gate="G$1" pin="GPIO11"/>
-<wire x1="45.72" y1="76.2" x2="55.88" y2="76.2" width="0.1524" layer="91"/>
-<label x="50.8" y="76.2" size="1.778" layer="95"/>
-</segment>
-</net>
-<net name="CS" class="0">
-<segment>
-<pinref part="J4" gate="G$1" pin="2"/>
-<wire x1="208.28" y1="35.56" x2="220.98" y2="35.56" width="0.1524" layer="91"/>
-<label x="213.36" y="35.56" size="1.778" layer="95"/>
-</segment>
-<segment>
-<pinref part="PCB1" gate="G$1" pin="GPIO8"/>
-<wire x1="17.78" y1="76.2" x2="7.62" y2="76.2" width="0.1524" layer="91"/>
-<label x="7.62" y="76.2" size="1.778" layer="95"/>
 </segment>
 </net>
@@
 </segment>
 <segment>
-<pinref part="PCB1" gate="G$1" pin="GPIO13"/>
-<wire x1="45.72" y1="101.6" x2="53.34" y2="101.6" width="0.1524" layer="91"/>
-<label x="50.8" y="101.6" size="1.778" layer="95"/>
+<pinref part="PCB1" gate="G$1" pin="GPIO27"/>
+<wire x1="45.72" y1="50.8" x2="55.88" y2="50.8" width="0.1524" layer="91"/>
+<label x="50.8" y="50.8" size="1.778" layer="95"/>
 </segment>
 </net>
@@
 <label x="238.76" y="137.16" size="1.778" layer="95"/>
 </segment>
+<segment>
+<pinref part="PCB1" gate="G$1" pin="GPIO22"/>
+<wire x1="45.72" y1="55.88" x2="55.88" y2="55.88" width="0.1524" layer="91"/>
+<label x="50.8" y="55.88" size="1.778" layer="95"/>
+</segment>
 </net>
 <net name="INT" class="0">
@@
 <net name="DI" class="0">
 <segment>
-<pinref part="PCB1" gate="G$1" pin="GPIO23"/>
-<wire x1="17.78" y1="55.88" x2="7.62" y2="55.88" width="0.1524" layer="91"/>
-<label x="7.62" y="55.88" size="1.778" layer="95"/>
-</segment>
-<segment>
 <pinref part="U$9" gate="G$1" pin="2"/>
 <wire x1="144.78" y1="15.24" x2="132.08" y2="15.24" width="0.1524" layer="91"/>
 <label x="132.08" y="15.24" size="1.778" layer="95"/>
 </segment>
+<segment>
+<pinref part="PCB1" gate="G$1" pin="GPIO16"/>
+<wire x1="17.78" y1="106.68" x2="7.62" y2="106.68" width="0.1524" layer="91"/>
+<label x="7.62" y="106.68" size="1.778" layer="95"/>
+</segment>
 </net>
 <net name="PI_POWER" class="0">
@@
 </segment>
 </net>
-<net name="IMU_NET" class="0">
-<segment>
-<pinref part="PCB1" gate="G$1" pin="GPIO6"/>
-<wire x1="45.72" y1="96.52" x2="53.34" y2="96.52" width="0.1524" layer="91"/>
-<label x="50.8" y="96.52" size="1.778" layer="95"/>
-</segment>
-</net>

Commit message: Minor Changes to Pi Shield
Parts:
- added R20: 4.7k, SparkFun-Resistors:RESISTOR0603
- added U$12: DF13-3P-1.25DSA, con-hirose-df13:DF13-3P-1.25DSA
Connections:
- new net PWM: PCB1.GPIO12, U$12.2
- net 5V: now also R20.2, U$12.1
- net DI: now also PCB1.GPIO21, R20.1; no longer PCB1.GPIO16
- net GND: now also U$12.3
Other:
- note added: "CAN Controller"
- note added: "CAN Termination"
- note added: "CAN Transceiver"
- note added: "Oscillator"
Changed lines of the file:
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@@
 <part name="C13" library="SparkFun-Capacitors" library_urn="urn:adsk.eagle:library:510" deviceset="22NF/22,000PF" device="-0603-50V-10%" package3d_urn="urn:adsk.eagle:package:37414@1/1" value=".1u"/>
 <part name="R19" library="SparkFun-Resistors" library_urn="urn:adsk.eagle:library:532" deviceset="RESISTOR" device="0603" package3d_urn="urn:adsk.eagle:package:39650/1" value="0"/>
+<part name="R20" library="SparkFun-Resistors" library_urn="urn:adsk.eagle:library:532" deviceset="RESISTOR" device="0603" package3d_urn="urn:adsk.eagle:package:39650/1" value="4.7k"/>
+<part name="U$12" library="con-hirose-df13" deviceset="DF13-3P-1.25" device="DSA"/>
 </parts>
 <sheets>
@@
 <plain>
 <text x="213.36" y="50.8" size="1.778" layer="91">NMOS</text>
+<text x="45.72" y="149.86" size="1.778" layer="91">CAN Controller</text>
+<text x="137.16" y="152.4" size="1.778" layer="91">CAN Transceiver</text>
+<text x="35.56" y="81.28" size="1.778" layer="91">Oscillator</text>
+<text x="200.66" y="154.94" size="1.778" layer="91">CAN Termination</text>
 </plain>
 <instances>
@@
 <text x="205.74" y="111.76" size="1.778" layer="91">External Power Supply Connectors</text>
 <text x="129.54" y="157.48" size="1.778" layer="91">LED to Indicate Power is ON</text>
-<text x="127" y="25.4" size="1.778" layer="91">Potential Temperature Sensor Connector</text>
+<text x="127" y="33.02" size="1.778" layer="91">Potential Temperature Sensor Connector</text>
 <text x="172.72" y="106.68" size="1.778" layer="91">Power Supply Connectors</text>
 </plain>
@@
 <instance part="U$9" gate="G$1" x="149.86" y="15.24"/>
 <instance part="C13" gate="G$1" x="231.14" y="160.02" rot="R90"/>
+<instance part="R20" gate="G$1" x="124.46" y="22.86" rot="R90"/>
+<instance part="U$12" gate="G$1" x="185.42" y="55.88"/>
 </instances>
 <busses>
@@
 <wire x1="144.78" y1="12.7" x2="132.08" y2="12.7" width="0.1524" layer="91"/>
 <label x="132.08" y="12.7" size="1.778" layer="95"/>
+</segment>
+<segment>
+<pinref part="U$12" gate="G$1" pin="3"/>
+<wire x1="180.34" y1="53.34" x2="172.72" y2="53.34" width="0.1524" layer="91"/>
+<label x="170.18" y="53.34" size="1.778" layer="95"/>
 </segment>
 </net>
@@
 <wire x1="144.78" y1="17.78" x2="132.08" y2="17.78" width="0.1524" layer="91"/>
 <label x="132.08" y="17.78" size="1.778" layer="95"/>
+<pinref part="R20" gate="G$1" pin="2"/>
+<wire x1="124.46" y1="27.94" x2="124.46" y2="30.48" width="0.1524" layer="91"/>
+<wire x1="124.46" y1="30.48" x2="132.08" y2="30.48" width="0.1524" layer="91"/>
+<wire x1="132.08" y1="30.48" x2="132.08" y2="17.78" width="0.1524" layer="91"/>
+</segment>
+<segment>
+<pinref part="U$12" gate="G$1" pin="1"/>
+<wire x1="180.34" y1="58.42" x2="172.72" y2="58.42" width="0.1524" layer="91"/>
+<label x="170.18" y="58.42" size="1.778" layer="95"/>
 </segment>
 </net>
@@
 <wire x1="144.78" y1="15.24" x2="132.08" y2="15.24" width="0.1524" layer="91"/>
 <label x="132.08" y="15.24" size="1.778" layer="95"/>
-</segment>
-<segment>
-<pinref part="PCB1" gate="G$1" pin="GPIO16"/>
-<wire x1="17.78" y1="106.68" x2="7.62" y2="106.68" width="0.1524" layer="91"/>
-<label x="7.62" y="106.68" size="1.778" layer="95"/>
+<wire x1="132.08" y1="15.24" x2="124.46" y2="15.24" width="0.1524" layer="91"/>
+<pinref part="R20" gate="G$1" pin="1"/>
+<wire x1="124.46" y1="15.24" x2="124.46" y2="17.78" width="0.1524" layer="91"/>
+</segment>
+<segment>
+<pinref part="PCB1" gate="G$1" pin="GPIO21"/>
+<wire x1="17.78" y1="116.84" x2="7.62" y2="116.84" width="0.1524" layer="91"/>
+<label x="7.62" y="116.84" size="1.778" layer="95"/>
 </segment>
 </net>
@@
 </segment>
 </net>
+<net name="PWM" class="0">
+<segment>
+<pinref part="U$12" gate="G$1" pin="2"/>
+<wire x1="180.34" y1="55.88" x2="172.72" y2="55.88" width="0.1524" layer="91"/>
+<label x="170.18" y="55.88" size="1.778" layer="95"/>
+</segment>
+<segment>
+<pinref part="PCB1" gate="G$1" pin="GPIO12"/>
+<wire x1="17.78" y1="96.52" x2="7.62" y2="96.52" width="0.1524" layer="91"/>
+<label x="7.62" y="96.52" size="1.778" layer="95"/>
+</segment>
+</net>

Commit message: Added Connectors, need to route
Parts:
- added J1, J2: (no value), SparkFun-Connectors:CONN_04
- added J6, J7: (no value), SparkFun-Connectors:CONN_02
- added U$13, U$14: T2I, BackplaneParts:T2I
- R1: value 10k -> 1k
- R10: value 47 -> 1k
- R2: value 1k -> 10k
Connections:
- removed net N$6: D1.A, R10.2
- new net AIN2: J2.2, U1.AIN2
- new net DI1: PCB1.GPIO16, U$14.3
- new net DI2: PCB1.GPIO20, U$14.2
- new net DI3: PCB1.GPIO21, U$14.1
- new net RESET_TO_PI: R10.2
- net 3V3: now also J1.4, J2.3, J6.2, J7.2
- net 5V: now also J2.4
- net CANH: now also U$13.2
- net CANL: now also U$13.3
- net DI: no longer PCB1.GPIO21
- net GND: now also J1.1, J2.1, J6.1, J7.1, U$14.4
- net N$3: now also D1.A
- net SCL: now also J1.2
- net SDA: now also J1.3
Other:
- note added: "3.3V Header Connectors"
- note added: "Additional Analog Input Sensor"
- note added: "CAN to MiniROV Connectors"
- note added: "Data Logger Pin"
- note added: "Possible Additional Sensor"
- moved on the sheet: C4, D1, D2, Q4, R1, R10, R2, R4, R5
